File: electrical/sbc_board/sbc_upd7220vga/sbc_upd7220vga.sch (KiCad schematic (older format))
At the start: 5 parts

Commit message: Kicad schematic capture
still need JTAG for CPLD but otherwise I think it's complete. PCB netlist load passes.
Parts:
- added C1: 22pF, Capacitor_SMD:C_0805_2012Metric_Pad1.18x1.45mm_HandSolder, symbol Device:C_Small
- added C10, C11, C12, C13, C5, C7, C8, C9: 1uF, Capacitor_SMD:C_0805_2012Metric_Pad1.18x1.45mm_HandSolder, symbol Device:C_Small
- added C14, C15, C16, C17, C18, C6: 10nF, Capacitor_SMD:C_0805_2012Metric_Pad1.18x1.45mm_HandSolder, symbol Device:C_Small
- added C2, C3, C4: 22uF, Capacitor_SMD:C_0805_2012Metric_Pad1.18x1.45mm_HandSolder, symbol Device:C_Small
- added D1: BAV99, Package_TO_SOT_SMD:SOT-23_Handsoldering, symbol Device:D_Schottky_x2_Serial_AKC
- added H1, H2, H3, H4: MountingHole, MountingHole:MountingHole_4.3mm_M4, symbol Mechanical:MountingHole
- added J1: DEBUG, Connector_PinHeader_2.54mm:PinHeader_1x08_P2.54mm_Vertical, symbol Connector_Generic:Conn_01x08
- added J4, J5: GND, Connector_PinHeader_2.54mm:PinHeader_1x02_P2.54mm_Vertical, symbol Connector_Generic:Conn_01x02
- added L1: 2.2uH, Inductor_SMD:L_Taiyo-Yuden_NR-30xx_HandSoldering, symbol Device:L
- added R1, R2, R3, R4, R5: 270, Resistor_SMD:R_0805_2012Metric_Pad1.20x1.40mm_HandSolder, symbol Device:R_Small
- added R6, R8: 220K, Resistor_SMD:R_0805_2012Metric_Pad1.20x1.40mm_HandSolder, symbol Device:R_Small
- added R7: 62K, Resistor_SMD:R_0805_2012Metric_Pad1.20x1.40mm_HandSolder, symbol Device:R_Small
- added RN1, RN2, RN3: 270, Resistor_SMD:R_Array_Concave_4x0603, symbol Device:R_Pack04
- added TP1: CLK50, TestPoint:TestPoint_Plated_Hole_D2.0mm, symbol Connector:TestPoint_Small
- added TP2: RED, TestPoint:TestPoint_Plated_Hole_D2.0mm, symbol Connector:TestPoint_Small
- added TP3: GREEN, TestPoint:TestPoint_Plated_Hole_D2.0mm, symbol Connector:TestPoint_Small
- added TP4: BLUE, TestPoint:TestPoint_Plated_Hole_D2.0mm, symbol Connector:TestPoint_Small
- added TP5: W2XCLK, TestPoint:TestPoint_Plated_Hole_D2.0mm, symbol Connector:TestPoint_Small
- added TP6: PCLK, TestPoint:TestPoint_Plated_Hole_D2.0mm, symbol Connector:TestPoint_Small
- added TP7: PIXEL, TestPoint:TestPoint_Plated_Hole_D2.0mm, symbol Connector:TestPoint_Small
- added TP8: VDD, TestPoint:TestPoint_Plated_Hole_D2.0mm, symbol Connector:TestPoint_Small
- added TP9: SEL, TestPoint:TestPoint_Plated_Hole_D2.0mm, symbol Connector:TestPoint_Small
- added U2: 71V016, Package_SO:TSOP-II-44_10.16x18.41mm_P0.8mm, symbol sbc_upd7220:71V016
- added U4: 74CB3T3245, Package_SO:TSSOP-20_4.4x6.5mm_P0.65mm, symbol 74xx:74LS245
- added U5: UPD7220, Package_DIP:DIP-40_W15.24mm, symbol sbc_upd7220:UPD7220
- added U6, U9: 74LVC245, Package_SO:TSSOP-20_4.4x6.5mm_P0.65mm, symbol 74xx:74LS245
- added U7: 74LVC574, Package_SO:TSSOP-20_4.4x6.5mm_P0.65mm, symbol 74xx:74LS574
- added U8: AP3429A, Package_TO_SOT_SMD:SOT-23-5, symbol Regulator_Switching:TLV62568DBV
- added X1: 50MHz, Oscillator:Oscillator_SMD_Abracon_ASV-4Pin_7.0x5.1mm, symbol Oscillator:ASV-xxxMHz
- J2: renamed from J?; footprint (none) -> Connector_PinHeader_2.54mm:PinHeader_2x20_P2.54mm_Vertical
- J3: renamed from J?; footprint (none) -> Connector_Dsub:DSUB-15-HD_Female_Horizontal_P2.29x2.54mm_EdgePinOffset9.40mm
- U1: renamed from U?; footprint (none) -> Package_SO:TSSOP-20_4.4x6.5mm_P0.65mm
- gave numbers to parts that had none: 1
Connections:
- net A17: now reaches U3.1 (IO1_1)
- net A17: now also U6.18 (B0)
- net GND: now reaches U3.10 (GNDIO)
- net GND: now also J2.37 (Pin_37), J2.38 (Pin_38), J2.39 (Pin_39), J2.40 (Pin_40), J3.10, J3.5, J3.6, J3.7, J3.8, U1.10 (GND), U3.115 (GNDIO), U3.128 (GNDINT), U3.135 (GNDIO), U3.17 (GNDINT), U3.26 (GNDIO), U3.47 (GNDIO), U3.54 (GNDINT), U3.65 (GNDIO), U3.83 (GNDIO), U3.92 (GNDINT), U3.99 (GNDIO), C10.2, C11.2, C12.2, C13.2, C14.2, C15.2, C16.2, C17.2, C18.2, C2.2, C3.2, C4.2, C5.2, C6.2, C7.2, C8.2, C9.2, J4.1 (Pin_1), J4.2 (Pin_2), J5.1 (Pin_1), J5.2 (Pin_2), R7.2, R8.2, RN1.3 (R3.1), RN1.4 (R4.1), RN2.3 (R3.1), RN2.4 (R4.1), RN3.3 (R3.1), RN3.4 (R4.1), U2.12 (VSS), U2.34 (VSS), U4.10 (GND), U5.20 (GND), U5.21 (LPEN), U6.10 (GND), U6.19 (CE), U7.1 (OE), U7.10 (GND), U8.2 (GND), U9.10 (GND), U9.19 (CE), X1.2 (GND)
- net PCLK: now reaches U3.109 (IO2_109)
- net PCLK: now also TP6.1, U7.11 (Cp)
- net R1OUT: now reaches U3.110 (IO2_110)
- net R1OUT: now also U7.2 (D0)
- net R0OUT: now reaches U3.111 (IO2_111)
- net R0OUT: now also U7.3 (D1)
- net G1OUT: now reaches U3.112 (IO2_112)
- net G1OUT: now also U7.4 (D2)
- net G0OUT: now reaches U3.113 (IO2_113)
- net G0OUT: now also U7.5 (D3)
- net B1OUT: now reaches U3.114 (IO2_114)
- net B1OUT: now also U7.6 (D4)
- net +3V3: now reaches U3.116 (VCCIO2)
- net +3V3: now also U1.20 (VCC), U3.100 (VCCIO3), U3.126 (VCCINT), U3.136 (VCCIO2), U3.19 (VCCINT), U3.25 (VCCIO1), U3.46 (VCCIO4), U3.56 (VCCINT), U3.64 (VCCIO4), U3.82 (VCCIO3), U3.9 (VCCIO1), U3.90 (VCCINT), C1.1, C10.1, C11.1, C12.1, C13.1, C14.1, C15.1, C16.1, C17.1, C18.1, C3.1, C4.1, C7.1, C8.1, C9.1, L1.2, R6.1, TP8.1, U2.11 (VDD), U2.33 (VDD), U4.20 (VCC), U6.1 (A->B), U6.20 (VCC), U7.20 (VCC), U9.1 (A->B), U9.20 (VCC), X1.1 (EN), X1.4 (Vdd)
- net B0OUT: now reaches U3.117 (IO2_117)
- net B0OUT: now also U7.7 (D5)
- net HSOUT: now reaches U3.118 (IO2_118)
- net HSOUT: now also U7.8 (D6)
- net VSOUT: now reaches U3.119 (IO2_119)
- net VSOUT: now also U7.9 (D7)
- net PIXEL: now reaches U3.120 (IO2_120)
- net PIXEL: now also TP7.1
- net DBG0: now reaches U3.137 (IO2_137)
- net DBG0: now also J1.1 (Pin_1)
- net DBG1: now reaches U3.138 (IO2_138)
- net DBG1: now also J1.2 (Pin_2)
- net DBG2: now reaches U3.139 (IO2_139)
- net DBG2: now also J1.3 (Pin_3)
- net DBG3: now reaches U3.140 (IO2_140)
- net DBG3: now also J1.4 (Pin_4)
- net DBG4: now reaches U3.141 (IO2_141)
- net DBG4: now also J1.5 (Pin_5)
- net DBG5: now reaches U3.142 (IO2_142)
- net DBG5: now also J1.6 (Pin_6)
- net DBG6: now reaches U3.143 (IO2_143)
- net DBG6: now also J1.7 (Pin_7)
- net DBG7: now reaches U3.144 (IO2_144)
- net DBG7: now also J1.8 (Pin_8)
- net GWR: now reaches U3.15 (IO1_15)
- net GWR: now also U5.10 (~WR)
- net GRD: now reaches U3.16 (IO1_16)
- net GRD: now also U5.9 (~RD)
- net CLK50: now reaches U3.18 (IO1_18/GCLK0)
- net CLK50: now also TP1.1, X1.3 (OUT)
- net A16: now reaches U3.2 (IO1_2)
- net A16: now also U6.17 (B1)
- net W2XCLK: now reaches U3.20 (IO1_20/GCLK1)
- net W2XCLK: now also TP5.1, U5.1 (W2XCLK)
- net HWR: now reaches U3.21 (IO1_21)
- net HWR: now also U9.18 (B0)
- net HRD: now reaches U3.22 (IO1_22)
- net HRD: now also U9.17 (B1)
- net HA3: now reaches U3.23 (IO1_23)
- net HA3: now also U9.16 (B2)
- net HA4: now reaches U3.24 (IO1_24)
- net HA4: now also U9.15 (B3)
- net HA5: now reaches U3.27 (IO1_27)
- net HA5: now also U9.14 (B4)
- net HA6: now reaches U3.28 (IO1_28)
- net HA6: now also U9.13 (B5)
- net HA7: now reaches U3.29 (IO1_29)
- net HA7: now also U9.12 (B6)
- net ALE: now reaches U3.3 (IO1_3)
- net ALE: now also U6.16 (B2)
- net HIOSEL: now reaches U3.30 (IO1_30)
- net HIOSEL: now also TP9.1, U9.11 (B7)
- net VBHE: now reaches U3.31 (IO1_31)
- net VBHE: now also U2.40 (~BHE)
- net VBLE: now reaches U3.32 (IO1_32)
- net VBLE: now also U2.39 (~BLE)
- net DBIN: now reaches U3.4 (IO1_4)
- net DBIN: now also U6.15 (B3)
- net HS: now reaches U3.5 (IO1_5)
- net HS: now also J3.13, R4.1, U6.14 (B4)
- net VS: now reaches U3.6 (IO1_6)
- net VS: now also J3.14, R5.1, U6.13 (B5)
- net BLANK: now reaches U3.7 (IO1_7)
- net BLANK: now also U6.12 (B6)
- net AD0: now reaches U3.37 (IO4_37)
- net AD0: now also U1.11 (B7), U2.7 (DQ0)
- net AD1: now reaches U3.38 (IO4_38)
- net AD1: now also U1.12 (B6), U2.8 (DQ1)
- net AD2: now reaches U3.39 (IO4_39)
- net AD2: now also U1.13 (B5), U2.9 (DQ2)
- net AD3: now reaches U3.40 (IO4_40)
- net AD3: now also U1.14 (B4), U2.10 (DQ3)
- net AD4: now reaches U3.41 (IO4_41)
- net AD4: now also U1.15 (B3), U2.13 (DQ4)
- net AD5: now reaches U3.42 (IO4_42)
- net AD5: now also U1.16 (B2), U2.14 (DQ5)
- net AD6: now reaches U3.43 (IO4_43)
- net AD6: now also U1.17 (B1), U2.15 (DQ6)
- net AD7: now reaches U3.44 (IO4_44)
- net AD7: now also U1.18 (B0), U2.16 (DQ7)
- net AD8: now reaches U3.45 (IO4_45)
- net AD8: now also U2.29 (DQ8), U4.11 (B7)
- net AD9: now reaches U3.48 (IO4_48)
- net AD9: now also U2.30 (DQ9), U4.12 (B6)
- net AD10: now reaches U3.49 (IO4_49)
- net AD10: now also U2.31 (DQ10), U4.13 (B5)
- net AD11: now reaches U3.50 (IO4_50)
- net AD11: now also U2.32 (DQ11), U4.14 (B4)
- net AD12: now reaches U3.51 (IO4_51)
- net AD12: now also U2.35 (DQ12), U4.15 (B3)
- net AD13: now reaches U3.52 (IO4_52)
- net AD13: now also U2.36 (DQ13), U4.16 (B2)
- net AD14: now reaches U3.53 (IO4_53)
- net AD14: now also U2.37 (DQ14), U4.17 (B1)
- net AD15: now reaches U3.55 (IO4_55)
- net AD15: now also U2.38 (DQ15), U4.18 (B0)
- net VCE: now reaches U3.57 (IO4_57)
- net VCE: now also U2.6 (~CE)
- net VOE: now reaches U3.58 (IO4_58)
- net VOE: now also U2.41 (~OE)
- net VWE: now reaches U3.59 (IO4_59)
- net VWE: now also U2.17 (~WE)
- net CPLD_RES: now reaches U3.61 (IO4_61/DEV_CLRn)
- net CPLD_RES: now also U6.11 (B7)
- net VA0: now reaches U3.62 (IO4_62)
- net VA0: now also U2.5 (A0)
- net VA1: now reaches U3.63 (IO4_63)
- net VA1: now also U2.4 (A1)
- net VA2: now reaches U3.66 (IO4_66)
- net VA2: now also U2.3 (A2)
- net VA3: now reaches U3.67 (IO4_67)
- net VA3: now also U2.2 (A3)
- net VA4: now reaches U3.68 (IO4_68)
- net VA4: now also U2.1 (A4)
- net VA5: now reaches U3.69 (IO4_69)
- net VA5: now also U2.44 (A5)
- net VA6: now reaches U3.70 (IO4_70)
- net VA6: now also U2.43 (A6)
- net VA7: now reaches U3.71 (IO4_71)
- net VA7: now also U2.42 (A7)
- net VA8: now reaches U3.72 (IO4_72)
- net VA8: now also U2.27 (A8)
- net VA9: now reaches U3.73 (IO3_73)
- net VA9: now also U2.26 (A9)
- net VA10: now reaches U3.74 (IO3_74)
- net VA10: now also U2.25 (A10)
- net VA11: now reaches U3.75 (IO3_75)
- net VA11: now also U2.24 (A11)
- net VA12: now reaches U3.76 (IO3_76)
- net VA12: now also U2.21 (A12)
- net VA13: now reaches U3.77 (IO3_77)
- net VA13: now also U2.20 (A13)
- net VA14: now reaches U3.78 (IO3_78)
- net VA14: now also U2.19 (A14)
- net VA15: now reaches U3.79 (IO3_79)
- net VA15: now also U2.18 (A15)
- net GDPEN: now reaches U1.19 (CE)
- net GDPEN: now also U4.19 (CE)
- net GAD7: now reaches U1.2 (A0)
- net GAD7: now also U5.29 (AD7)
- net GAD6: now reaches U1.3 (A1)
- net GAD6: now also U5.28 (AD6)
- net GAD5: now reaches U1.4 (A2)
- net GAD5: now also U5.27 (AD5)
- net GAD4: now reaches U1.5 (A3)
- net GAD4: now also U5.26 (AD4)
- net GAD3: now reaches U1.6 (A4)
- net GAD3: now also U5.25 (AD3)
- net GAD2: now reaches U1.7 (A5)
- net GAD2: now also U5.24 (AD2)
- net GAD1: now reaches U1.8 (A6)
- net GAD1: now also U5.23 (AD1)
- net GAD0: now reaches U1.9 (A7)
- net GAD0: now also U5.22 (AD0)
- net VCC: now reaches J2.1 (Pin_1)
- net VCC: now also J2.2 (Pin_2), J2.3 (Pin_3), J2.4 (Pin_4), J3.9, C2.1, C5.1, C6.1, U5.40 (VCC), U8.1 (EN), U8.4 (VIN)
- net A6: now reaches J2.11 (Pin_11)
- net A6: now also U9.7 (A5)
- net A5: now reaches J2.13 (Pin_13)
- net A5: now also U9.6 (A4)
- net A4: now reaches J2.15 (Pin_15)
- net A4: now also U9.5 (A3)
- net A3: now reaches J2.17 (Pin_17)
- net A3: now also U9.4 (A2)
- net RD: now reaches J2.18 (Pin_18)
- net RD: now also U9.3 (A1)
- net A0: now reaches J2.23 (Pin_23)
- net A0: now also U5.11 (A0)
- net D7: now reaches J2.24 (Pin_24)
- net D7: now also U5.19 (D7)
- net D0: now reaches J2.25 (Pin_25)
- net D0: now also U5.12 (D0)
- net D6: now reaches J2.26 (Pin_26)
- net D6: now also U5.18 (D6)
- net D1: now reaches J2.27 (Pin_27)
- net D1: now also U5.13 (D1)
- net D5: now reaches J2.28 (Pin_28)
- net D5: now also U5.17 (D5)
- net D2: now reaches J2.29 (Pin_29)
- net D2: now also U5.14 (D2)
- net D4: now reaches J2.30 (Pin_30)
- net D4: now also U5.16 (D4)
- net IOSEL: now reaches J2.31 (Pin_31)
- net IOSEL: now also U9.9 (A7)
- net D3: now reaches J2.32 (Pin_32)
- net D3: now also U5.15 (D3)
- net RESET: now reaches J2.35 (Pin_35)
- net RESET: now also U6.9 (A7)
- net IRQ: now reaches J2.36 (Pin_36)
- net IRQ: now also D1.3 (common)
- net WR: now reaches J2.8 (Pin_8)
- net WR: now also U9.2 (A0)
- net A7: now reaches J2.9 (Pin_9)
- net A7: now also U9.8 (A6)
- net RED: now reaches J3.1
- net RED: now also RN1.5 (R4.2), RN1.6 (R3.2), RN1.7 (R2.2), RN1.8 (R1.2), TP2.1
- net GREEN: now reaches J3.2
- net GREEN: now also RN2.5 (R4.2), RN2.6 (R3.2), RN2.7 (R2.2), RN2.8 (R1.2), TP3.1
- net BLUE: now reaches J3.3
- net BLUE: now also RN3.5 (R4.2), RN3.6 (R3.2), RN3.7 (R2.2), RN3.8 (R1.2), TP4.1
- new net: R1.1, RN1.2 (R2.1)
- new net: R2.1, RN2.2 (R2.1)
- new net: R3.1, RN3.2 (R2.1)
- new net: L1.1, U8.3 (SW)
- new net: C1.2, R6.2, R7.1, R8.1, U8.5 (FB)
- new net B0Q: R3.2, U7.14 (Q5)
- new net B1Q: RN3.1 (R1.1), U7.15 (Q4)
- new net CPLD_IRQ: D1.2 (K)
- new net G0Q: R2.2, U7.16 (Q3)
- new net G1Q: RN2.1 (R1.1), U7.17 (Q2)
- new net GA16: U5.38 (A16), U6.3 (A1)
- new net GA17: U5.39 (A17), U6.2 (A0)
- new net GAD10: U4.7 (A5), U5.32 (AD10)
- new net GAD11: U4.6 (A4), U5.33 (AD11)
- new net GAD12: U4.5 (A3), U5.34 (AD12)
- new net GAD13: U4.4 (A2), U5.35 (AD13)
- new net GAD14: U4.3 (A1), U5.36 (AD14)
- new net GAD15: U4.2 (A0), U5.37 (AD15)
- new net GAD8: U4.9 (A7), U5.30 (AD8)
- new net GAD9: U4.8 (A6), U5.31 (AD9)
- new net GALE: U5.6 (ALE), U6.4 (A2)
- new net GBLANK: U5.5 (BLANK), U6.8 (A6)
- new net GDBIN: U5.2 (~DBIN), U6.5 (A3)
- new net GHS: U5.3 (HSYNC), U6.6 (A4)
- new net GVS: U5.4 (VSYNC), U6.7 (A5)
- new net HSQ: R4.2, U7.13 (Q6)
- new net R0Q: R1.2, U7.18 (Q1)
- new net R1Q: RN1.1 (R1.1), U7.19 (Q0)
- new net VSQ: R5.2, U7.12 (Q7)
- no-connect marks 0 -> 19
Other:
- moved on the sheet: J2, J3, U1, U3A, U3B
